File: ESP32/ESP32.kicad_pcb (KiCad board)
At the start: 2 copper layers, 68.6 x 40.6 mm, 2 parts, among them U1 ESP32-WROOM-32, U2 Generic_5v_Module

Commit message: KiCad Updates
Routing:
- net Net-(U1-Pad2): track 0.00 -> 106.6 mm
- net Net-(U1-Pad1): track 0.00 -> 92.9 mm
- net unconnected-(U2-Pad1): track 0.00 -> 2.54 mm
- net unconnected-(U2-Pad2): track 0.00 -> 2.54 mm
Changed lines of the file:
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@@
       (viasonmask false)
       (mode 1)
-      (useauxorigin false)
+      (useauxorigin true)
       (hpglpennumber 1)
       (hpglpenspeed 20)
@@
       (drillshape 0)
       (scaleselection 1)
-      (outputdirectory "")
+      (outputdirectory "./")
     )
   )
@@
       (effects (font (size 1 1) (thickness 0.15)))
     )
-    (fp_line (start 7.62 -7.62) (end 7.62 -5.08) (layer "F.SilkS") (width 0.12))
+    (fp_line (start -12.7 5.08) (end -12.7 -10.16) (layer "F.SilkS") (width 0.12))
+    (fp_line (start -12.7 -10.16) (end 10.16 -10.16) (layer "F.SilkS") (width 0.12))
     (fp_line (start 10.16 -10.16) (end 10.16 5.08) (layer "F.SilkS") (width 0.12))
-    (fp_line (start 7.62 0) (end 7.62 2.54) (layer "F.SilkS") (width 0.12))
-    (fp_line (start 7.62 -7.62) (end 7.62 -5.08) (layer "F.SilkS") (width 0.12))
-    (fp_line (start -10.16 0) (end -10.16 2.54) (layer "F.SilkS") (width 0.12))
-    (fp_line (start -10.16 -7.62) (end -10.16 -5.08) (layer "F.SilkS") (width 0.12))
-    (fp_line (start -12.7 -10.16) (end 10.16 -10.16) (layer "F.SilkS") (width 0.12))
     (fp_line (start 10.16 5.08) (end -12.7 5.08) (layer "F.SilkS") (width 0.12))
-    (fp_line (start -12.7 5.08) (end -12.7 -10.16) (layer "F.SilkS") (width 0.12))
+    (pad "1" thru_hole circle (at -10.16 -5.08) (size 1.524 1.524) (drill 0.762) (layers *.Cu *.Mask)
+      (net 37 "unconnected-(U2-Pad1)") (pinfunction "IN+") (pintype "input+no_connect"))
     (pad "1" thru_hole circle (at -10.16 -7.62) (size 1.524 1.524) (drill 0.762) (layers *.Cu *.Mask)
       (net 37 "unconnected-(U2-Pad1)") (pinfunction "IN+") (pintype "input+no_connect"))
-    (pad "1" thru_hole circle (at -10.16 -5.08) (size 1.524 1.524) (drill 0.762) (layers *.Cu *.Mask)
-      (net 37 "unconnected-(U2-Pad1)") (pinfunction "IN+") (pintype "input+no_connect"))
+    (pad "2" thru_hole circle (at -10.16 2.54) (size 1.524 1.524) (drill 0.762) (layers *.Cu *.Mask)
+      (net 38 "unconnected-(U2-Pad2)") (pinfunction "IN-") (pintype "input+no_connect"))
     (pad "2" thru_hole circle (at -10.16 0) (size 1.524 1.524) (drill 0.762) (layers *.Cu *.Mask)
       (net 38 "unconnected-(U2-Pad2)") (pinfunction "IN-") (pintype "input+no_connect"))
-    (pad "2" thru_hole circle (at -10.16 2.54) (size 1.524 1.524) (drill 0.762) (layers *.Cu *.Mask)
-      (net 38 "unconnected-(U2-Pad2)") (pinfunction "IN-") (pintype "input+no_connect"))
+    (pad "3" thru_hole circle (at 7.62 -7.62) (size 1.524 1.524) (drill 0.762) (layers *.Cu *.Mask)
+      (net 2 "Net-(U1-Pad2)") (pinfunction "5v") (pintype "output"))
     (pad "3" thru_hole circle (at 7.62 -5.08) (size 1.524 1.524) (drill 0.762) (layers *.Cu *.Mask)
-      (net 2 "Net-(U1-Pad2)") (pinfunction "5v") (pintype "output"))
-    (pad "3" thru_hole circle (at 7.62 -7.62) (size 1.524 1.524) (drill 0.762) (layers *.Cu *.Mask)
       (net 2 "Net-(U1-Pad2)") (pinfunction "5v") (pintype "output"))
     (pad "4" thru_hole circle (at 7.62 2.54) (size 1.524 1.524) (drill 0.762) (layers *.Cu *.Mask)
@@
   )
   (gr_rect (start 124.46 88.9) (end 193.04 129.54) (layer "Edge.Cuts") (width 0.1) (fill none))
+  (segment (start 144.145 106.045) (end 147.027989 108.927989) (width 0.25) (layer "F.Cu") (net 1))
+  (segment (start 157.48 124.46) (end 180.34 124.46) (width 0.25) (layer "F.Cu") (net 1))
+  (segment (start 147.027989 108.927989) (end 149.910978 106.045) (width 0.25) (layer "F.Cu") (net 1))
+  (segment (start 149.910978 106.045) (end 150.74 106.045) (width 0.25) (layer "F.Cu") (net 1))
+  (segment (start 150.74 106.045) (end 151.99 106.045) (width 0.25) (layer "F.Cu") (net 1))
+  (segment (start 157.48 111.535) (end 157.48 124.46) (width 0.25) (layer "F.Cu") (net 1))
+  (segment (start 180.34 124.46) (end 185.42 119.38) (width 0.25) (layer "F.Cu") (net 1))
+  (segment (start 133.74 106.045) (end 144.145 106.045) (width 0.25) (layer "F.Cu") (net 1))
+  (segment (start 185.42 119.38) (end 185.42 116.84) (width 0.25) (layer "F.Cu") (net 1))
+  (segment (start 151.99 106.045) (end 157.48 111.535) (width 0.25) (layer "F.Cu") (net 1))
+  (segment (start 136.525 119.430978) (end 147.027989 108.927989) (width 0.25) (layer "F.Cu") (net 1))
+  (segment (start 136.525 123.555) (end 136.525 119.430978) (width 0.25) (layer "F.Cu") (net 1))
+  (segment (start 185.42 109.22) (end 185.42 111.76) (width 0.25) (layer "F.Cu") (net 2))
+  (segment (start 133.74 107.315) (end 132.49 107.315) (width 0.25) (layer "F.Cu") (net 2))
+  (segment (start 190.5 127) (end 190.5 116.84) (width 0.25) (layer "F.Cu") (net 2))
+  (segment (start 132.49 107.315) (end 127 112.805) (width 0.25) (layer "F.Cu") (net 2))
+  (segment (start 127 112.805) (end 127 127) (width 0.25) (layer "F.Cu") (net 2))
+  (segment (start 190.5 116.84) (end 185.42 111.76) (width 0.25) (layer "F.Cu") (net 2))
+  (segment (start 127 127) (end 190.5 127) (width 0.25) (layer "F.Cu") (net 2))
+  (segment (start 167.64 109.22) (end 167.64 111.76) (width 0.25) (layer "F.Cu") (net 37))
+  (segment (start 167.64 116.84) (end 167.64 119.38) (width 0.25) (layer "F.Cu") (net 38))
 )

Commit message: KiCad Changes.
Parts:
- added J1: Screw_Terminal_01x02, TerminalBlock:TerminalBlock_bornier-2_P5.08mm, F.Cu at (147.3, 91.4)
- added J2: Screw_Terminal_01x02, TerminalBlock:TerminalBlock_bornier-2_P5.08mm, F.Cu at (158.9, 91.4)
- added Q1: IRLZ44N, Package_TO_SOT_THT:TO-220-3_Vertical, F.Cu at (149.9, 104.1)
- added R1: R_Small_US, Resistor_THT:R_Axial_DIN0207_L6.3mm_D2.5mm_P5.08mm_Vertical, F.Cu at (149.9, 111.8)
- U1: value ESP32-WROOM-32 -> NodeMCU_ESP8266_LUA_12-F; footprint RF_Module:ESP32-WROOM-32 -> ESP32_modules:NodeMCU 8266 LUA 12-F
- moved U1 18.2 mm to (130.8, 100.2)
Connections:
- U1 pad 1: Net-(U1-Pad1) -> unconnected-(U1-Pad1)
- U1 pad 10: unconnected-(U1-Pad10) -> GND
- U1 pad 11: Net-(R1-Pad1) -> unconnected-(U1-Pad11)
- U1 pad 15: Net-(U1-Pad1) -> +5V
- U1 pad 18: unconnected-(U1-Pad18) -> ENABLE
- U1 pad 2: Net-(U1-Pad2) -> unconnected-(U1-Pad2)
- U1 pad 22: unconnected-(U1-Pad22) -> GND
- U1 pad 29: unconnected-(U1-Pad29) -> GND
- U2 pad 1: unconnected-(U2-Pad1) -> VCC
- U2 pad 2: unconnected-(U2-Pad2) -> GND
- U2 pad 3: Net-(U1-Pad2) -> +5V
- U2 pad 4: Net-(U1-Pad1) -> GND
Routing:
- net Net-(U1-Pad2): track 106.6 -> 0.00 mm
- net Net-(U1-Pad1): track 92.9 -> 0.00 mm
- net GND: track 0.00 -> 5.08 mm
- net unconnected-(U2-Pad1): track 2.54 -> 0.00 mm
- net VCC: track 0.00 -> 2.54 mm
- net +5V: track 0.00 -> 2.54 mm
- net unconnected-(U2-Pad2): track 2.54 -> 0.00 mm
Other:
- board size 68.6 x 40.6 mm -> 73.7 x 50.8 mm
