File: ESP32/ESP32.kicad_sch (KiCad schematic)
At the start: 4 parts, among them Q1 Q_NPN_EBC, U1 ESP32-WROOM-32, U2 Generic_5v_Module

Commit message: KiCad Updates
Parts:
- removed U1: ESP32-WROOM-32, RF_Module:ESP32-WROOM-32, symbol RF_Module:ESP32-WROOM-32
- added U?: ESP32, ESP32_modules:ESP32-DevKitC, symbol Espressif:ESP32
Other:
- moved on the sheet: U2
Changed lines of the file:
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@@
   (no_connect (at 181.61 85.09))
   (no_connect (at 181.61 90.17))
-  (wire (pts (xy 201.93 43.18) (xy 201.93 85.09))
+  (wire (pts (xy 204.47 43.18) (xy 204.47 85.09))
     (stroke (width 0) (type default) (color 0 0 0 0))
   )
@@
     (stroke (width 0) (type default) (color 0 0 0 0))
   )
-  (wire (pts (xy 137.16 43.18) (xy 201.93 43.18))
+  (wire (pts (xy 137.16 43.18) (xy 204.47 43.18))
     (stroke (width 0) (type default) (color 0 0 0 0))
   )
@@
     (stroke (width 0) (type default) (color 0 0 0 0))
   )
-  (symbol (lib_id "RF_Module:ESP32-WROOM-32") (at 137.16 86.36 0) (unit 1)
+  (symbol (lib_id "power:GND") (at 193.04 114.3 0) (unit 1)
     (in_bom yes) (on_board yes) (fields_autoplaced)
-    (property "Reference" "U1" (id 0) (at 139.1794 48.26 0)
+    (property "Reference" "#PWR02" (id 0) (at 193.04 120.65 0)
+      (effects (font (size 1.27 1.27)) hide)
+    )
+    (property "Value" "GND" (id 1) (at 193.04 119.38 0))
+    (property "Footprint" "" (id 2) (at 193.04 114.3 0)
+      (effects (font (size 1.27 1.27)) hide)
+    )
+    (property "Datasheet" "" (id 3) (at 193.04 114.3 0)
+      (effects (font (size 1.27 1.27)) hide)
+    )
+    (pin "1")
+  )
+  (symbol (lib_id "Device:Q_NPN_EBC") (at 190.5 104.14 0) (unit 1)
+    (in_bom yes) (on_board yes) (fields_autoplaced)
+    (property "Reference" "Q1" (id 0) (at 195.58 102.8699 0)
       (effects (font (size 1.27 1.27)) (justify left))
     )
-    (property "Value" "ESP32-WROOM-32" (id 1) (at 139.1794 50.8 0)
+    (property "Value" "Q_NPN_EBC" (id 1) (at 195.58 105.4099 0)
       (effects (font (size 1.27 1.27)) (justify left))
     )
-    (property "Footprint" "RF_Module:ESP32-WROOM-32" (id 2) (at 137.16 124.46 0)
+    (property "Footprint" "" (id 2) (at 195.58 101.6 0)
       (effects (font (size 1.27 1.27)) hide)
     )
-    (property "Datasheet" "https://www.espressif.com/sites/default/files/documentation/esp32-wroom-32_datasheet_en.pdf" (id 3) (at 129.54 85.09 0)
+    (property "Datasheet" "~" (id 3) (at 190.5 104.14 0)
+      (effects (font (size 1.27 1.27)) hide)
+    )
+    (pin "1")
+    (pin "2")
+    (pin "3")
+  )
+  (symbol (lib_id "Espressif:ESP32") (at 86.36 95.25 0) (unit 1)
+    (in_bom yes) (on_board yes) (fields_autoplaced)
+    (property "Reference" "U?" (id 0) (at 86.995 48.26 0))
+    (property "Value" "ESP32" (id 1) (at 86.995 50.8 0))
+    (property "Footprint" "ESP32_modules:ESP32-DevKitC" (id 2) (at 92.71 88.9 0)
+      (effects (font (size 1.27 1.27)) hide)
+    )
+    (property "Datasheet" "https://www.espressif.com/sites/default/files/documentation/esp32_datasheet_en.pdf" (id 3) (at 92.71 88.9 0)
       (effects (font (size 1.27 1.27)) hide)
     )
@@
     (pin "39")
     (pin "4")
+    (pin "40")
+    (pin "41")
+    (pin "42")
+    (pin "43")
+    (pin "44")
+    (pin "45")
+    (pin "46")
+    (pin "47")
+    (pin "48")
+    (pin "49")
     (pin "5")
     (pin "6")
@@
     (pin "8")
     (pin "9")
-  )
-  (symbol (lib_id "power:GND") (at 193.04 114.3 0) (unit 1)
-    (in_bom yes) (on_board yes) (fields_autoplaced)
-    (property "Reference" "#PWR02" (id 0) (at 193.04 120.65 0)
-      (effects (font (size 1.27 1.27)) hide)
-    )
-    (property "Value" "GND" (id 1) (at 193.04 119.38 0))
-    (property "Footprint" "" (id 2) (at 193.04 114.3 0)
-      (effects (font (size 1.27 1.27)) hide)
-    )
-    (property "Datasheet" "" (id 3) (at 193.04 114.3 0)
-      (effects (font (size 1.27 1.27)) hide)
-    )
-    (pin "1")
-  )
-  (symbol (lib_id "Device:Q_NPN_EBC") (at 190.5 104.14 0) (unit 1)
-    (in_bom yes) (on_board yes) (fields_autoplaced)
-    (property "Reference" "Q1" (id 0) (at 195.58 102.8699 0)
-      (effects (font (size 1.27 1.27)) (justify left))
-    )
-    (property "Value" "Q_NPN_EBC" (id 1) (at 195.58 105.4099 0)
-      (effects (font (size 1.27 1.27)) (justify left))
-    )
-    (property "Footprint" "" (id 2) (at 195.58 101.6 0)
-      (effects (font (size 1.27 1.27)) hide)
-    )
-    (property "Datasheet" "~" (id 3) (at 190.5 104.14 0)
-      (effects (font (size 1.27 1.27)) hide)
-    )
-    (pin "1")
-    (pin "2")
-    (pin "3")
   )
   (symbol (lib_id "Converter_DCDC:Generic_5v_Module") (at 184.15 82.55 0) (unit 1)
@@
       (reference "R1") (unit 1) (value "R_Small_US") (footprint "")
     )
-    (path "/01c54f9e-832d-4b6f-a713-b99706de04cd"
-      (reference "U1") (unit 1) (value "ESP32-WROOM-32") (footprint "RF_Module:ESP32-WROOM-32")
-    )
     (path "/af686684-ac69-4d50-b35e-6e5471573a3e"
       (reference "U2") (unit 1) (value "Generic_5v_Module") (footprint "Converter_DCDC:DCDC_Generic-5v")
     )
+    (path "/74ca8f24-2a26-45b7-bd7a-6213e5f96148"
+      (reference "U?") (unit 1) (value "ESP32") (footprint "ESP32_modules:ESP32-DevKitC")
+    )
   )

Commit message: KiCad Changes.
Parts:
- removed Q1: Q_NPN_EBC, symbol Device:Q_NPN_EBC
- removed U?: ESP32, ESP32_modules:ESP32-DevKitC, symbol Espressif:ESP32
- added J1, J2: Screw_Terminal_01x02, TerminalBlock:TerminalBlock_bornier-2_P5.08mm, symbol Connector:Screw_Terminal_01x02
- added Q1: IRLZ44N, Package_TO_SOT_THT:TO-220-3_Vertical, symbol Transistor_FET:IRLZ44N
- added U1: NodeMCU_ESP8266_LUA_12-F, ESP32_modules:NodeMCU 8266 LUA 12-F, symbol Espressif:NodeMCU_ESP8266_LUA_12-F
- R1: footprint (none) -> Resistor_THT:R_Axial_DIN0207_L6.3mm_D2.5mm_P5.08mm_Vertical
Connections:
- net GND: now also U2.2 (IN-), U2.4 (5v-), J2.2 (Pin_2), Q1.3 (S), U1.10 (GND0), U1.22 (GND2), U1.29 (GND3)
- net at R1.2: now also Q1.1 (G)
- net VCC: now reaches U2.1 (IN+)
- net VCC: now also J1.1 (Pin_1), J2.1 (Pin_1)
- net +5V: now reaches U2.3 (5v)
- net +5V: now also U1.15 (VIN)
- net ENABLE: now reaches R1.1
- net ENABLE: now also U1.18 (D2)
- new net MOSFET_GND: J1.2 (Pin_2), Q1.2 (D)
- no-connect marks 3 -> 22
