File: 8266_NODEMCU_ESP12F/ESP32.kicad_pcb (KiCad board)
At the start: 2 copper layers, 73.7 x 50.8 mm, 6 parts, among them J1 Screw_Terminal_01x02, J2 Screw_Terminal_01x02, Q1 IRLZ44N, U1 NodeMCU_ESP8266_LUA_12-F, U2 Generic_5v_Module

Commit message: KiCad Updates
Routing:
- net GND: track 5.08 -> 97.0 mm
- net +5V: track 2.54 -> 72.8 mm
- net VCC: track 2.54 -> 44.8 mm
- net ENABLE: track 0.00 -> 21.4 mm
- net MOSFET_GND: track 0.00 -> 12.5 mm
- net Net-(R1-Pad2): track 0.00 -> 9.72 mm
Changed lines of the file:
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@@
       (usegerberattributes true)
       (usegerberadvancedattributes true)
-      (creategerberjobfile true)
+      (creategerberjobfile false)
       (svguseinch false)
       (svgprecision 6)
@@
       (drillshape 0)
       (scaleselection 1)
-      (outputdirectory "./")
+      (outputdirectory "Gerber/")
     )
   )
@@
     )
   )
+  (gr_line (start 167.64 116.84) (end 167.64 119.38) (layer "F.Cu") (width 0.2))
   (gr_rect (start 116.84 83.82) (end 190.5 134.62) (layer "Edge.Cuts") (width 0.1) (fill none))
+  (segment (start 149.86 88.9) (end 156.33 88.9) (width 0.25) (layer "F.Cu") (net 1))
+  (segment (start 158.87 91.44) (end 161.41 88.9) (width 0.25) (layer "F.Cu") (net 1))
+  (segment (start 167.64 91.44) (end 167.64 109.22) (width 0.25) (layer "F.Cu") (net 1))
+  (segment (start 161.41 88.9) (end 165.1 88.9) (width 0.25) (layer "F.Cu") (net 1))
+  (segment (start 156.33 88.9) (end 158.87 91.44) (width 0.25) (layer "F.Cu") (net 1))
+  (segment (start 165.1 88.9) (end 167.64 91.44) (width 0.25) (layer "F.Cu") (net 1))
+  (segment (start 147.32 91.44) (end 149.86 88.9) (width 0.25) (layer "F.Cu") (net 1))
   (segment (start 167.64 109.22) (end 167.64 111.76) (width 0.25) (layer "F.Cu") (net 1))
+  (segment (start 152.4 103.539639) (end 152.099819 103.83982) (width 0.25) (layer "F.Cu") (net 2))
+  (segment (start 152.4 91.44) (end 152.4 103.539639) (width 0.25) (layer "F.Cu") (net 2))
+  (segment (start 138.445 105.255) (end 133.365 105.255) (width 0.25) (layer "F.Cu") (net 10))
+  (segment (start 147.32 114.3) (end 149.93071 114.3) (width 0.25) (layer "F.Cu") (net 10))
+  (segment (start 167.21548 116.664159) (end 167.33982 116.539819) (width 0.25) (layer "F.Cu") (net 10))
   (segment (start 167.64 116.84) (end 167.64 119.38) (width 0.25) (layer "F.Cu") (net 10))
+  (segment (start 155.240181 107.970119) (end 163.934221 116.664159) (width 0.25) (layer "F.Cu") (net 10))
+  (segment (start 149.93071 114.3) (end 155.240181 108.990529) (width 0.25) (layer "F.Cu") (net 10))
+  (segment (start 163.95 95.130001) (end 155.240181 103.83982) (width 0.25) (layer "F.Cu") (net 10))
+  (segment (start 138.445 123.035) (end 135.905 123.035) (width 0.25) (layer "F.Cu") (net 10))
+  (segment (start 138.445 105.255) (end 138.445 105.425) (width 0.25) (layer "F.Cu") (net 10))
+  (segment (start 138.445 105.425) (end 147.32 114.3) (width 0.25) (layer "F.Cu") (net 10))
+  (segment (start 163.95 91.44) (end 163.95 95.130001) (width 0.25) (layer "F.Cu") (net 10))
   (segment (start 185.42 119.38) (end 185.42 116.84) (width 0.25) (layer "F.Cu") (net 10))
+  (segment (start 135.905 123.035) (end 125.745 112.875) (width 0.25) (layer "F.Cu") (net 10))
+  (segment (start 133.365 105.255) (end 125.745 112.875) (width 0.25) (layer "F.Cu") (net 10))
+  (segment (start 163.934221 116.664159) (end 167.21548 116.664159) (width 0.25) (layer "F.Cu") (net 10))
+  (segment (start 155.240181 107.970119) (end 155.24018 104.44018) (width 0.25) (layer "F.Cu") (net 10))
+  (segment (start 155.240181 108.990529) (end 155.240181 107.970119) (width 0.25) (layer "F.Cu") (net 10))
+  (segment (start 170.18 129.54) (end 129.54 129.54) (width 0.25) (layer "F.Cu") (net 26))
+  (segment (start 129.54 129.54) (end 129.54 129.37) (width 0.25) (layer "F.Cu") (net 26))
   (segment (start 185.42 109.22) (end 185.42 111.76) (width 0.25) (layer "F.Cu") (net 26))
+  (segment (start 129.54 129.37) (end 125.745 125.575) (width 0.25) (layer "F.Cu") (net 26))
+  (segment (start 185.42 111.76) (end 185.42 114.3) (width 0.25) (layer "F.Cu") (net 26))
+  (segment (start 185.42 114.3) (end 170.18 129.54) (width 0.25) (layer "F.Cu") (net 26))
+  (segment (start 142.24 104.06929) (end 149.86 111.68929) (width 0.25) (layer "F.Cu") (net 29))
+  (segment (start 142.24 98.89) (end 142.24 104.06929) (width 0.25) (layer "F.Cu") (net 29))
+  (segment (start 149.86 111.68929) (end 149.86 111.76) (width 0.25) (layer "F.Cu") (net 29))
+  (segment (start 138.445 95.095) (end 142.24 98.89) (width 0.25) (layer "F.Cu") (net 29))
+  (segment (start 149.86 106.68) (end 154.94 111.76) (width 0.25) (layer "B.Cu") (net 31))
+  (segment (start 149.86 104.14) (end 149.86 106.68) (width 0.25) (layer "B.Cu") (net 31))
 )

Commit message: PCB updates
Parts:
- added J3: Screw_Terminal_01x02, TerminalBlock:TerminalBlock_bornier-2_P5.08mm, F.Cu at (182.9, 127.0)
- added J4: Screw_Terminal_01x02, TerminalBlock:TerminalBlock_bornier-2_P5.08mm, F.Cu at (182.9, 114.3)
- added J5: Screw_Terminal_01x03, TerminalBlock:TerminalBlock_bornier-3_P5.08mm, F.Cu at (172.7, 88.9)
- added RV1: R_Potentiometer_Trim_US, Potentiometer_THT:Potentiometer_Runtron_RM-065_Vertical, F.Cu at (127.0, 106.7)
- added SW1: SW_SPDT, Button_Switch_THT:SW_DIP_SPSTx01_Slide_6.7x4.1mm_W7.62mm_P2.54mm_LowProfile, F.Cu at (176.5, 101.6)
- U2: value Generic_5v_Module -> DC-DC Buck
- moved U2 50.0 mm to (132.1, 96.5)
- moved J2 49.7 mm to (127.0, 129.5), turned to 180 degrees
- moved J1 38.9 mm to (139.7, 129.5), turned to 180 degrees
- moved Q1 25.1 mm to (132.1, 121.9), turned to 90 degrees
- moved U1 24.1 mm to (154.9, 99.1)
- moved R1 22.9 mm to (172.7, 111.8), turned to -90 degrees
Connections:
- J1 pad 2: MOSFET_GND -> Variable Ground
- U1 pad 24: unconnected-(U1-Pad24) -> PUL
- U1 pad 25: unconnected-(U1-Pad25) -> DIR
- U1 pad 5: unconnected-(U1-Pad5) -> Net-(U1-Pad5)
Routing:
- net Variable Ground: track 0.00 -> 84.4 mm
- net Net-(U1-Pad5): track 0.00 -> 72.7 mm
- net GND: track 97.0 -> 161.4 mm
- net MOSFET_GND: track 12.5 -> 51.8 mm
- net Net-(Q1-Pad1): track 9.72 -> 42.7 mm
- net DIR: track 0.00 -> 26.6 mm
- net PUL: track 0.00 -> 22.4 mm
- net ENABLE: track 21.4 -> 39.3 mm
- net +5V: track 72.8 -> 87.2 mm
- net VCC: track 44.8 -> 57.0 mm
Other:
- board text added: "5V"
