File: 8266_NODEMCU_ESP12F/ESP32.kicad_sch (KiCad schematic)
At the start: 6 parts, among them J1 Screw_Terminal_01x02, J2 Screw_Terminal_01x02, Q1 IRLZ44N, U1 NodeMCU_ESP8266_LUA_12-F, U2 Generic_5v_Module

Commit message: KiCad Updates
Parts:
- added SW?: SW_SPDT, symbol Switch:SW_SPDT
Other:
- moved on the sheet: J1, J2, Q1, R1, U1, U2

Commit message: PCB updates
Parts:
- added J3, J4: Screw_Terminal_01x02, TerminalBlock:TerminalBlock_bornier-2_P5.08mm, symbol Connector:Screw_Terminal_01x02
- added J5: Screw_Terminal_01x03, TerminalBlock:TerminalBlock_bornier-3_P5.08mm, symbol Connector:Screw_Terminal_01x03
- added RV1: R_Potentiometer_Trim_US, Potentiometer_THT:Potentiometer_Runtron_RM-065_Vertical, symbol Device:R_Potentiometer_Trim_US
- gave numbers to parts that had none: 1
Connections:
- net +5V: now also J5.1 (Pin_1), RV1.1
- net ENABLE: now also J5.2 (Pin_2)
- net GND: now also SW1.3 (C), J3.2 (Pin_2), J4.2 (Pin_2), J5.3 (Pin_3), RV1.3
- net MOSFET_GND: now also SW1.1 (A); no longer J1.2 (Pin_2)
- net PUL: now reaches U1.24 (D6)
- net PUL: now also J4.1 (Pin_1)
- net DIR: now reaches U1.25 (D7)
- net DIR: now also J3.1 (Pin_1)
- net at U1.5 (SD2): now also RV1.2
- net Variable Ground: now reaches SW1.2 (B)
- net Variable Ground: now also J1.2 (Pin_2)
- no-connect marks 22 -> 18
Other:
- moved on the sheet: U1
