File: 8266_NODEMCU_ESP12F/8266.kicad_sch (KiCad schematic)
At the start: 11 parts, among them J1 Screw_Terminal_01x02, J2 Screw_Terminal_01x02, J3 Screw_Terminal_01x02, J4 Screw_Terminal_01x02, J5 Screw_Terminal_01x03, Q1 IRLZ44N, SW1 SW_SPDT, U1 NodeMCU_ESP8266_LUA_12-F, U2 Generic_5v_Module

Commit message: PCB changes agian
Parts:
- added H1, H2, H3: MountingHole, MountingHole:MountingHole_3.2mm_M3, symbol Mechanical:MountingHole
- R1: value R_Small_US -> 10k
- SW1: footprint (none) -> Button_Switch_THT:Slide Switch
Changed lines of the file:
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@@
     (pin "3")
   )
+  (symbol (lib_id "Mechanical:MountingHole") (at 232.41 26.67 0) (unit 1)
+    (in_bom yes) (on_board yes) (fields_autoplaced)
+    (property "Reference" "H1" (id 0) (at 234.95 25.3999 0)
+      (effects (font (size 1.27 1.27)) (justify left))
+    )
+    (property "Value" "MountingHole" (id 1) (at 234.95 27.9399 0)
+      (effects (font (size 1.27 1.27)) (justify left))
+    )
+    (property "Footprint" "MountingHole:MountingHole_3.2mm_M3" (id 2) (at 232.41 26.67 0)
+      (effects (font (size 1.27 1.27)) hide)
+    )
+    (property "Datasheet" "~" (id 3) (at 232.41 26.67 0)
+      (effects (font (size 1.27 1.27)) hide)
+    )
+  )
   (symbol (lib_id "Switch:SW_SPDT") (at 226.06 55.88 0) (unit 1)
-    (in_bom yes) (on_board yes) (fields_autoplaced)
+    (in_bom yes) (on_board yes)
     (property "Reference" "SW1" (id 0) (at 226.06 48.26 0))
     (property "Value" "SW_SPDT" (id 1) (at 226.06 50.8 0))
-    (property "Footprint" "" (id 2) (at 226.06 55.88 0)
-      (effects (font (size 1.27 1.27)) hide)
-    )
+    (property "Footprint" "Button_Switch_THT:Slide Switch" (id 2) (at 229.87 66.04 0))
     (property "Datasheet" "~" (id 3) (at 226.06 55.88 0)
       (effects (font (size 1.27 1.27)) hide)
@@
     )
     (pin "1")
+  )
+  (symbol (lib_id "Mechanical:MountingHole") (at 250.19 31.75 0) (unit 1)
+    (in_bom yes) (on_board yes) (fields_autoplaced)
+    (property "Reference" "H3" (id 0) (at 252.73 30.4799 0)
+      (effects (font (size 1.27 1.27)) (justify left))
+    )
+    (property "Value" "MountingHole" (id 1) (at 252.73 33.0199 0)
+      (effects (font (size 1.27 1.27)) (justify left))
+    )
+    (property "Footprint" "MountingHole:MountingHole_3.2mm_M3" (id 2) (at 250.19 31.75 0)
+      (effects (font (size 1.27 1.27)) hide)
+    )
+    (property "Datasheet" "~" (id 3) (at 250.19 31.75 0)
+      (effects (font (size 1.27 1.27)) hide)
+    )
   )
   (symbol (lib_id "Connector:Screw_Terminal_01x02") (at 127 173.99 0) (unit 1)
@@
     (pin "1")
   )
+  (symbol (lib_id "Mechanical:MountingHole") (at 250.19 24.13 0) (unit 1)
+    (in_bom yes) (on_board yes) (fields_autoplaced)
+    (property "Reference" "H2" (id 0) (at 252.73 22.8599 0)
+      (effects (font (size 1.27 1.27)) (justify left))
+    )
+    (property "Value" "MountingHole" (id 1) (at 252.73 25.3999 0)
+      (effects (font (size 1.27 1.27)) (justify left))
+    )
+    (property "Footprint" "MountingHole:MountingHole_3.2mm_M3" (id 2) (at 250.19 24.13 0)
+      (effects (font (size 1.27 1.27)) hide)
+    )
+    (property "Datasheet" "~" (id 3) (at 250.19 24.13 0)
+      (effects (font (size 1.27 1.27)) hide)
+    )
+  )
   (symbol (lib_id "Connector:Screw_Terminal_01x02") (at 232.41 142.24 0) (unit 1)
     (in_bom yes) (on_board yes) (fields_autoplaced)
@@
     (in_bom yes) (on_board yes) (fields_autoplaced)
     (property "Reference" "R1" (id 0) (at 223.52 118.11 90))
-    (property "Value" "R_Small_US" (id 1) (at 223.52 120.65 90))
+    (property "Value" "10k" (id 1) (at 223.52 120.65 90))
     (property "Footprint" "Resistor_THT:R_Axial_DIN0207_L6.3mm_D2.5mm_P5.08mm_Vertical" (id 2) (at 223.52 124.46 0)
       (effects (font (size 1.27 1.27)) hide)
@@
       (reference "#PWR0105") (unit 1) (value "GND") (footprint "")
     )
+    (path "/4f6e05b4-9880-489a-8124-b7f416144db1"
+      (reference "H1") (unit 1) (value "MountingHole") (footprint "MountingHole:MountingHole_3.2mm_M3")
+    )
+    (path "/de184e78-e5be-4119-938c-56c55936e4bc"
+      (reference "H2") (unit 1) (value "MountingHole") (footprint "MountingHole:MountingHole_3.2mm_M3")
+    )
+    (path "/8b338a1a-27a6-4b2f-9828-da95f534b845"
+      (reference "H3") (unit 1) (value "MountingHole") (footprint "MountingHole:MountingHole_3.2mm_M3")
+    )
     (path "/cf970825-c949-4581-abbc-10bd58d97e15"
       (reference "J1") (unit 1) (value "Screw_Terminal_01x02") (footprint "TerminalBlock:TerminalBlock_bornier-2_P5.08mm")
@@
     )
     (path "/e43aa29c-427c-47ef-9d4b-7a062511150f"
-      (reference "R1") (unit 1) (value "R_Small_US") (footprint "Resistor_THT:R_Axial_DIN0207_L6.3mm_D2.5mm_P5.08mm_Vertical")
+      (reference "R1") (unit 1) (value "10k") (footprint "Resistor_THT:R_Axial_DIN0207_L6.3mm_D2.5mm_P5.08mm_Vertical")
     )
     (path "/02376529-a7f0-4ee0-82d0-c26b2b59531d"
@@
     )
     (path "/54e869da-5e86-4640-b5b1-e8da3b8b993d"
-      (reference "SW1") (unit 1) (value "SW_SPDT") (footprint "")
+      (reference "SW1") (unit 1) (value "SW_SPDT") (footprint "Button_Switch_THT:Slide Switch")
     )
     (path "/1819a01d-5413-4f2e-bee3-b9f9334a34dc"

Commit message: Code changes, beta code and Schema changes.
Connections:
- net DIR: now also U1.18 (D2); no longer U1.25 (D7)
- net ENABLE: now also U1.24 (D6); no longer U1.18 (D2)
- net PUL: now also U1.19 (D3); no longer U1.24 (D6)
- no-connect marks 18 -> 19
Changed lines of the file:
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@@
   (no_connect (at 153.67 81.28))
   (no_connect (at 153.67 83.82))
-  (no_connect (at 153.67 88.9))
   (no_connect (at 153.67 91.44))
   (no_connect (at 153.67 93.98))
@@
   (no_connect (at 133.35 96.52))
   (no_connect (at 133.35 93.98))
+  (no_connect (at 153.67 104.14))
+  (no_connect (at 127 77.47))
   (wire (pts (xy 213.36 55.88) (xy 220.98 55.88))
     (stroke (width 0) (type default) (color 0 0 0 0))
   )
-  (wire (pts (xy 153.67 101.6) (xy 162.56 101.6))
-    (stroke (width 0) (type default) (color 0 0 0 0))
-  )
   (wire (pts (xy 231.14 53.34) (xy 242.57 53.34))
     (stroke (width 0) (type default) (color 0 0 0 0))
@@
     (stroke (width 0) (type default) (color 0 0 0 0))
   )
-  (wire (pts (xy 153.67 104.14) (xy 162.56 104.14))
+  (wire (pts (xy 153.67 86.36) (xy 157.48 86.36))
     (stroke (width 0) (type default) (color 0 0 0 0))
   )
@@
     (stroke (width 0) (type default) (color 0 0 0 0))
   )
-  (wire (pts (xy 153.67 86.36) (xy 161.29 86.36))
-    (stroke (width 0) (type default) (color 0 0 0 0))
-  )
   (wire (pts (xy 118.11 90.17) (xy 120.65 90.17))
     (stroke (width 0) (type default) (color 0 0 0 0))
@@
     (stroke (width 0) (type default) (color 0 0 0 0))
   )
+  (wire (pts (xy 153.67 88.9) (xy 157.48 88.9))
+    (stroke (width 0) (type default) (color 0 0 0 0))
+  )
   (wire (pts (xy 120.65 90.17) (xy 120.65 87.63))
     (stroke (width 0) (type default) (color 0 0 0 0))
@@
     (stroke (width 0) (type default) (color 0 0 0 0))
   )
+  (wire (pts (xy 153.67 101.6) (xy 157.48 101.6))
+    (stroke (width 0) (type default) (color 0 0 0 0))
+  )
   (wire (pts (xy 210.82 124.46) (xy 220.98 124.46))
     (stroke (width 0) (type default) (color 0 0 0 0))
@@
     )
   )
-  (global_label "DIR" (shape input) (at 162.56 104.14 0) (fields_autoplaced)
-    (effects (font (size 1.27 1.27)) (justify left))
-    (property "Intersheet References" "${INTERSHEET_REFS}" (id 0) (at 168.1179 104.0606 0)
+  (global_label "DIR" (shape input) (at 157.48 86.36 0) (fields_autoplaced)
+    (effects (font (size 1.27 1.27)) (justify left))
+    (property "Intersheet References" "${INTERSHEET_REFS}" (id 0) (at 163.0379 86.2806 0)
       (effects (font (size 1.27 1.27)) (justify left) hide)
     )
@@
     )
   )
-  (global_label "ENABLE" (shape input) (at 161.29 86.36 0) (fields_autoplaced)
-    (effects (font (size 1.27 1.27)) (justify left))
-    (property "Intersheet References" "${INTERSHEET_REFS}" (id 0) (at 170.7183 86.4394 0)
+  (global_label "ENABLE" (shape input) (at 157.48 101.6 0) (fields_autoplaced)
+    (effects (font (size 1.27 1.27)) (justify left))
+    (property "Intersheet References" "${INTERSHEET_REFS}" (id 0) (at 166.9083 101.6794 0)
       (effects (font (size 1.27 1.27)) (justify left) hide)
     )
@@
     )
   )
-  (global_label "PUL" (shape input) (at 162.56 101.6 0) (fields_autoplaced)
-    (effects (font (size 1.27 1.27)) (justify left))
-    (property "Intersheet References" "${INTERSHEET_REFS}" (id 0) (at 168.6017 101.5206 0)
+  (global_label "PUL" (shape input) (at 157.48 88.9 0) (fields_autoplaced)
+    (effects (font (size 1.27 1.27)) (justify left))
+    (property "Intersheet References" "${INTERSHEET_REFS}" (id 0) (at 163.5217 88.8206 0)
       (effects (font (size 1.27 1.27)) (justify left) hide)
     )
@@
   )
   (symbol (lib_id "power:GND") (at 158.75 96.52 90) (unit 1)
-    (in_bom yes) (on_board yes) (fields_autoplaced)
+    (in_bom yes) (on_board yes)
     (property "Reference" "#PWR04" (id 0) (at 165.1 96.52 0)
       (effects (font (size 1.27 1.27)) hide)
     )
-    (property "Value" "GND" (id 1) (at 162.56 96.5199 90)
-      (effects (font (size 1.27 1.27)) (justify right))
-    )
+    (property "Value" "GND" (id 1) (at 157.48 83.8199 90)
+      (effects (font (size 1.27 1.27)) (justify right))
+    )
