File: esp32/_autosave-NodeMCU-32S.kicad_pcb (KiCad board)
At the start: 2 copper layers, 87 x 71.1 mm, 16 parts, among them J1 Screw_Terminal_01x02, J2 Screw_Terminal_01x02, J3 Screw_Terminal_01x02, J4 Screw_Terminal_01x02, J5 Screw_Terminal_01x03, Q1 IRLZ44N, SW1 SW_SPST, U1 ESP32-DevKitC, U2 Generic_5v_Module

Commit message: Version 1.4
Sliding Switch & C++ code changeds.
Other:
- board text added: "Board Design 1.4"
Changed lines of the file:
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@@
   (gr_line (start 119.2022 90.0176) (end 116.6622 92.5576) (layer "F.SilkS") (width 0.15))
   (gr_rect (start 58 45.6692) (end 145.034 116.7892) (layer "Edge.Cuts") (width 0.2) (fill none))
+  (gr_text "Board Design 1.4" (at 88.8746 52.2732) (layer "B.SilkS")
+    (effects (font (size 3 3) (thickness 0.25)) (justify mirror))
+  )
   (gr_text "-" (at 139.7 76.2 90) (layer "F.SilkS")
     (effects (font (size 1 1) (thickness 0.15)))
@@
     (effects (font (size 1 1) (thickness 0.15)))
   )
-  (gr_text "CCW" (at 138.7094 101.9048) (layer "F.SilkS")
+  (gr_text "CCW" (at 138.7094 101.9048 90) (layer "F.SilkS")
     (effects (font (size 1 1) (thickness 0.15)))
   )
-  (gr_text "CW" (at 138.303 96.4692) (layer "F.SilkS")
+  (gr_text "CW" (at 138.303 96.4692 90) (layer "F.SilkS")
     (effects (font (size 1 1) (thickness 0.15)))
   )
