File: PCB Design/TTS Design.kicad_sch (KiCad schematic)
At the start: 22 parts, among them J1 Screw_Terminal_01x02, J2 Screw_Terminal_01x02, J3 Screw_Terminal_01x04, J5 Screw_Terminal_01x03, Q1 IRLZ44N, SW1 SW_DPDT_x2, SW2 SW_DPDT_x2, U1 ESP32-DevKitC, U2 Generic_5v_Module

Commit message: Board changes -- Diode
Parts:
- removed C2: C, Capacitor_THT:C_Disc_D3.0mm_W1.6mm_P2.50mm, symbol Device:C
Connections:
- net GND: no longer D1.1 (K), J2.2 (Pin_2)
- new net GNDPWR: D1.1 (K), J2.2 (Pin_2)
Changed lines of the file:
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@@
   (junction (at 193.04 121.92) (diameter 0) (color 0 0 0 0)
   )
-  (junction (at 76.2 19.05) (diameter 0) (color 0 0 0 0)
-  )
   (junction (at 100.33 144.78) (diameter 0) (color 0 0 0 0)
   )
   (junction (at 100.33 132.08) (diameter 0) (color 0 0 0 0)
-  )
-  (junction (at 76.2 26.67) (diameter 0) (color 0 0 0 0)
   )
   (no_connect (at 106.68 129.54))
@@
     (stroke (width 0) (type default))
   )
-  (wire (pts (xy 76.2 19.05) (xy 81.28 19.05))
-    (stroke (width 0) (type default))
-  )
   (wire (pts (xy 176.53 101.6) (xy 180.34 101.6))
     (stroke (width 0) (type default))
@@
     (stroke (width 0) (type default))
   )
-  (wire (pts (xy 62.23 19.05) (xy 76.2 19.05))
+  (wire (pts (xy 62.23 19.05) (xy 81.28 19.05))
     (stroke (width 0) (type default))
   )
@@
     (stroke (width 0) (type default))
   )
-  (wire (pts (xy 76.2 26.67) (xy 62.23 26.67))
-    (stroke (width 0) (type default))
-  )
   (wire (pts (xy 262.89 76.2) (xy 262.89 77.47))
     (stroke (width 0) (type default))
@@
     (stroke (width 0) (type default))
   )
-  (wire (pts (xy 76.2 26.67) (xy 81.28 26.67))
+  (wire (pts (xy 62.23 26.67) (xy 81.28 26.67))
     (stroke (width 0) (type default))
   )
@@
     )
   )
-  (symbol (lib_id "power:GND") (at 24.13 20.32 270) (unit 1)
-    (in_bom yes) (on_board yes) (dnp no) (fields_autoplaced)
-    (property "Reference" "#PWR06" (at 17.78 20.32 0)
-      (effects (font (size 1.27 1.27)) hide)
-    )
-    (property "Value" "GND" (at 20.32 20.3199 90)
-      (effects (font (size 1.27 1.27)) (justify right))
-    )
-    (property "Footprint" "" (at 24.13 20.32 0)
-      (effects (font (size 1.27 1.27)) hide)
-    )
-    (property "Datasheet" "" (at 24.13 20.32 0)
-      (effects (font (size 1.27 1.27)) hide)
-    )
-    (pin "1")
-    (instances
-      (project "TTS Design"
-        (path "/9dd029d7-3440-476c-a069-461d6098ced3"
-          (reference "#PWR06") (unit 1)
-        )
-      )
-    )
-  )
   (symbol (lib_id "Device:R_Potentiometer_Trim_US") (at 262.89 45.72 0) (unit 1)
     (in_bom yes) (on_board yes) (dnp no) (fields_autoplaced)
@@
     )
   )
-  (symbol (lib_id "Device:C") (at 76.2 22.86 0) (unit 1)
-    (in_bom yes) (on_board yes) (dnp no) (fields_autoplaced)
-    (property "Reference" "C2" (at 80.01 21.59 0)
-      (effects (font (size 1.27 1.27)) (justify left))
-    )
-    (property "Value" "C" (at 80.01 24.13 0)
-      (effects (font (size 1.27 1.27)) (justify left))
-    )
-    (property "Footprint" "Capacitor_THT:C_Disc_D3.0mm_W1.6mm_P2.50mm" (at 77.1652 26.67 0)
-      (effects (font (size 1.27 1.27)) hide)
-    )
-    (property "Datasheet" "~" (at 76.2 22.86 0)
-      (effects (font (size 1.27 1.27)) hide)
-    )
-    (pin "1")
-    (pin "2")
-    (instances
-      (project "TTS Design"
-        (path "/9dd029d7-3440-476c-a069-461d6098ced3"
-          (reference "C2") (unit 1)
-        )
-      )
-    )
-  )
   (symbol (lib_name "GND_1") (lib_id "power:GND") (at 81.28 19.05 90) (unit 1)
     (in_bom yes) (on_board yes) (dnp no) (fields_autoplaced)
@@
     )
   )
-  (symbol (lib_id "power:GND") (at 140.97 46.99 270) (unit 1)
-    (in_bom yes) (on_board yes) (dnp no) (fields_autoplaced)
-    (property "Reference" "#PWR09" (at 134.62 46.99 0)
-      (effects (font (size 1.27 1.27)) hide)
-    )
-    (property "Value" "GND" (at 137.16 46.9899 90)
-      (effects (font (size 1.27 1.27)) (justify right))
-    )
-    (property "Footprint" "" (at 140.97 46.99 0)
-      (effects (font (size 1.27 1.27)) hide)
-    )
-    (property "Datasheet" "" (at 140.97 46.99 0)
-      (effects (font (size 1.27 1.27)) hide)
-    )
-    (pin "1")
-    (instances
-      (project "TTS Design"
-        (path "/9dd029d7-3440-476c-a069-461d6098ced3"
-          (reference "#PWR09") (unit 1)
+  (symbol (lib_id "power:GNDPWR") (at 24.13 20.32 270) (unit 1)
+    (in_bom yes) (on_board yes) (dnp no) (fields_autoplaced)
+    (property "Reference" "#PWR06" (at 19.05 20.32 0)
+      (effects (font (size 1.27 1.27)) hide)
+    )
+    (property "Value" "GNDPWR" (at 20.32 20.193 90)
+      (effects (font (size 1.27 1.27)) (justify right))
+    )
+    (property "Footprint" "" (at 22.86 20.32 0)
+      (effects (font (size 1.27 1.27)) hide)
+    )
+    (property "Datasheet" "" (at 22.86 20.32 0)
+      (effects (font (size 1.27 1.27)) hide)
+    )
+    (pin "1")
+    (instances
+      (project "TTS Design"
+        (path "/9dd029d7-3440-476c-a069-461d6098ced3"
+          (reference "#PWR06") (unit 1)
         )
       )
@@
         )
       )
+    )
+  )
+  (symbol (lib_id "power:GNDPWR") (at 140.97 46.99 270) (unit 1)
+    (in_bom yes) (on_board yes) (dnp no) (fields_autoplaced)
+    (property "Reference" "#PWR08" (at 135.89 46.99 0)
+      (effects (font (size 1.27 1.27)) hide)
+    )
+    (property "Value" "GNDPWR" (at 137.16 46.863 90)
+      (effects (font (size 1.27 1.27)) (justify right))
+    )
+    (property "Footprint" "" (at 139.7 46.99 0)
+      (effects (font (size 1.27 1.27)) hide)
+    )
+    (property "Datasheet" "" (at 139.7 46.99 0)
+      (effects (font (size 1.27 1.27)) hide)
+    )
+    (pin "1")
+    (instances
+      (project "TTS Design"
+        (path "/9dd029d7-3440-476c-a069-461d6098ced3"
+          (reference "#PWR08") (unit 1)
+        )
+      )

Commit message: board changes
1 - larger through holes on DC Buck
2 - rerouted some tracks
Parts:
- added C2: C_Small, symbol Device:C_Small
Connections:
- net +5V: now also C2.2
- net GND: now also C2.1

Commit message: Board changes
Made Cap width larger, cleaned up dual pins on the MCU
Parts:
- C2: footprint (none) -> Capacitor_THT:C_Disc_D4.3mm_W1.9mm_P5.00mm
Changed lines of the file:
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@@
 			)
 		)
-		(property "Footprint" ""
+		(property "Footprint" "Capacitor_THT:C_Disc_D4.3mm_W1.9mm_P5.00mm"
 			(at 72.39 22.86 0)
 			(effects

Commit message: Through hole size change
footprint change
remaps connection
Parts:
- U2: footprint Converter_DCDC:DCDC_Generic-5v -> DC CUSTOM:DCDC_Generic-5v
Changed lines of the file:
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@@
 (kicad_sch
-	(version 20231120)
+	(version 20250114)
 	(generator "eeschema")
-	(generator_version "8.0")
+	(generator_version "9.0")
 	(paper "A4")
 	(title_block
@@
 			)
 		)
-		(property "Footprint" "Converter_DCDC:DCDC_Generic-5v"
+		(property "Footprint" "DC CUSTOM:DCDC_Generic-5v"
 			(at 36.83 17.78 0)
 			(effects
@@
 		)
 	)
+	(embedded_fonts no)
 )
